File: Schematics/555_Replacement/555_Replacement.kicad_sch (KiCad schematic)
At the start: 6 parts, among them SW1 Mode, SW2 "Step", U1 ATtiny85-20P

Commit message: Add files via upload
Parts:
- RV1: value "Cycle_Time" -> 10K
Connections:
- net GND: now also RV1.1; no longer RV1.3
- net VCC: now also RV1.3; no longer RV1.1
Other:
- moved on the sheet: RV1, SW1, SW2
